File: PCB/gate_output.kicad_sch (KiCad schematic)
At the start: 6 parts

Commit message: :sparkles: Add jack LEDs to the schematic
Using clear jacks the LEDs can be put underneath them. The control
PCB can support both versions (LEDs separate or in jacks), so a
second (SMD) LED is added to the schematic.

Only one of these may be populated!
Parts:
- added D?: gn, LED_SMD:LED_0805_2012Metric_Pad1.15x1.40mm_HandSolder, symbol Device:LED
Connections:
- net at D?.2 (A), Q?.3 (E), R?.2: now also D?.2 (A)
- net at D?.1 (K), R?.2: now also D?.1 (K)
Other:
- note added: "Adjust for SMD LED!"
- note added: "Only populate one LED!"
Changed lines of the file:
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@@
     (company "moPsy")
+  )
+  (junction (at 53.34 67.31) (diameter 0) (color 0 0 0 0)
+  )
+  (junction (at 53.34 55.245) (diameter 0) (color 0 0 0 0)
   )
   (junction (at 66.675 55.245) (diameter 0) (color 0 0 0 0)
@@
     (stroke (width 0) (type default))
   )
+  (wire (pts (xy 53.34 55.245) (xy 42.545 55.245))
+    (stroke (width 0) (type default))
+  )
   (polyline (pts (xy 40.005 43.18) (xy 37.465 43.18))
     (stroke (width 0) (type solid))
   )
+  (wire (pts (xy 53.34 67.31) (xy 53.34 69.85))
+    (stroke (width 0) (type default))
+  )
   (wire (pts (xy 82.55 69.85) (xy 82.55 71.12))
     (stroke (width 0) (type default))
@@
     (stroke (width 0) (type default))
   )
+  (wire (pts (xy 42.545 55.245) (xy 42.545 57.15))
+    (stroke (width 0) (type default))
+  )
   (wire (pts (xy 66.675 67.31) (xy 86.36 67.31))
     (stroke (width 0) (type default))
   )
+  (wire (pts (xy 42.545 64.77) (xy 42.545 67.31))
+    (stroke (width 0) (type default))
+  )
+  (wire (pts (xy 42.545 67.31) (xy 53.34 67.31))
+    (stroke (width 0) (type default))
+  )
   (wire (pts (xy 53.34 55.245) (xy 66.675 55.245))
     (stroke (width 0) (type default))
@@
     (stroke (width 0) (type default))
   )
-  (wire (pts (xy 53.34 64.77) (xy 53.34 69.85))
+  (wire (pts (xy 53.34 64.77) (xy 53.34 67.31))
     (stroke (width 0) (type default))
   )
@@
   (text "Output" (at 46.355 31.75 0)
     (effects (font (size 2.54 2.54)) (justify left bottom))
+  )
+  (text "Only populate\none LED!" (at 42.545 70.485 0)
+    (effects (font (size 0.8 0.8)) (justify left bottom))
+  )
+  (text "Adjust for\nSMD LED!" (at 55.88 78.74 0)
+    (effects (font (size 0.8 0.8)) (justify left bottom))
   )
   (hierarchical_label "GATE_OUT" (shape input) (at 41.275 45.72 180) (fields_autoplaced)
@@
         )
       )
+    )
+  )
+  (symbol (lib_id "Device:LED") (at 42.545 60.96 90) (unit 1)
+    (in_bom no) (on_board yes) (dnp yes)
+    (property "Reference" "D?" (at 46.355 60.96 90)
+      (effects (font (size 1.27 1.27)) (justify right))
+    )
+    (property "Value" "gn" (at 46.355 63.5 90)
+      (effects (font (size 1.27 1.27)) (justify right))
+    )
+    (property "Footprint" "LED_SMD:LED_0805_2012Metric_Pad1.15x1.40mm_HandSolder" (at 42.545 60.96 0)
+      (effects (font (size 1.27 1.27)) hide)
+    )
+    (property "Datasheet" "~" (at 42.545 60.96 0)
+      (effects (font (size 1.27 1.27)) hide)
+    )
+    (property "Sim.Enable" "0" (at 42.545 60.96 0)
+      (effects (font (size 1.27 1.27)) hide)
+    )
+    (property "REICHELT" "EVL 17-21SYGC" (at 42.545 60.96 90)
+      (effects (font (size 1.27 1.27)) hide)
+    )
+    (pin "1")
+    (pin "2")
+    (instances
+      (project "manual-gate-trigger-source"
+        (path "/64d6412c-bfad-42df-9ed7-bcc6cbff0470/5e147908-dd0e-44a6-bf7b-e0f4f3b88ce0"
+          (reference "D?") (unit 1)
+        )
+        (path "/64d6412c-bfad-42df-9ed7-bcc6cbff0470/4d130511-3de2-468d-9ad3-9fd4dd47645e"
+          (reference "D?") (unit 1)
+        )
+        (path "/64d6412c-bfad-42df-9ed7-bcc6cbff0470/b83b5c1b-da69-40b5-857e-949eb4f1eab8"
+          (reference "D?") (unit 1)
+        )
+        (path "/64d6412c-bfad-42df-9ed7-bcc6cbff0470/b0ca186f-8794-49d8-ae6e-2d447887c3e3"
+          (reference "D?") (unit 1)
+        )
+      )
+      (project "div"
+        (path "/69636855-5bea-4b1f-bae0-d5724c7c5e69"
+          (reference "D?") (unit 1)
+        )
+        (path "/69636855-5bea-4b1f-bae0-d5724c7c5e69/ddb23b62-aa27-4614-8e08-b908b2a2dd99"
+          (reference "D13") (unit 1)
+        )
+        (path "/69636855-5bea-4b1f-bae0-d5724c7c5e69/61f4bdd8-3e4f-4e0c-a5fa-951e97fb38b8"
+          (reference "D14") (unit 1)
+        )
+        (path "/69636855-5bea-4b1f-bae0-d5724c7c5e69/d48a94fa-bfe1-4bce-a3d7-937659f4df9e"
+          (reference "D15") (unit 1)
+        )
+        (path "/69636855-5bea-4b1f-bae0-d5724c7c5e69/e2f85f9a-c5ab-41b2-b8ce-b63f382b5258"
+          (reference "D16") (unit 1)
+        )
+        (path "/69636855-5bea-4b1f-bae0-d5724c7c5e69/301a9e1d-1dbb-4a63-a88b-1d93e257644e"
+          (reference "D17") (unit 1)
+        )
+        (path "/69636855-5bea-4b1f-bae0-d5724c7c5e69/82e60134-6463-4f35-8227-ac1dc3c9b002"
+          (reference "D18") (unit 1)
+        )
+      )

Commit message: :wrench: Adjust output resistor divider
Give a bit more driving power to the outputs by lowering the output
resistor divider.

This results in a current of 2.7mA through the resistor divider
or 5.5mA in case of a short circuit.

With all outputs switched on, consumption is 16.3mA
(32.7mA short ciruit).
Parts:
- R? (x2): value 4k7 -> 2k2
Changed lines of the file:
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@@
       (effects (font (size 1.27 1.27)) (justify right))
     )
-    (property "Value" "4k7" (at 69.215 62.5475 0)
+    (property "Value" "2k2" (at 69.215 62.5475 0)
       (effects (font (size 1.27 1.27)) (justify right))
     )
@@
       (effects (font (size 1.27 1.27)) (justify right))
     )
-    (property "Value" "4k7" (at 69.215 74.6125 0)
+    (property "Value" "2k2" (at 69.215 74.6125 0)
       (effects (font (size 1.27 1.27)) (justify right))
     )

Commit message: :wrench: Change transistor footprint to handsolder version
Parts:
- Q?: footprint Package_TO_SOT_THT:TO-92_Inline -> Package_TO_SOT_THT:TO-92_HandSolder
Changed lines of the file:
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@@
       (effects (font (size 1.27 1.27)) (justify left))
     )
-    (property "Footprint" "Package_TO_SOT_THT:TO-92_Inline" (at 69.215 47.625 0)
+    (property "Footprint" "Package_TO_SOT_THT:TO-92_HandSolder" (at 69.215 47.625 0)
       (effects (font (size 1.27 1.27) italic) (justify left) hide)
     )
