File: PCB/gate_output.kicad_sch (KiCad schematic)
At the start: 7 parts

Commit message: :wrench: Change LED footprint to 0603
This is harder to solder, but matching LEDs with 180mcd are available:
* https://www.reichelt.de/led-smd-1608-0603-rot-180-mcd-120--led-el-0603-rt-p156256.html
* https://www.reichelt.de/led-smd-1608-0603-gelb-180-mcd-120--led-el-0603-ge-p156259.html
Parts:
- D?: footprint LED_SMD:LED_0805_2012Metric_Pad1.15x1.40mm_HandSolder -> LED_SMD:LED_0603_1608Metric_Pad1.05x0.95mm_HandSolder
Other:
- note added: "180mcd or more"
- note removed: "Adjust for SMD LED!"
Changed lines of the file:
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@@
     (effects (font (size 0.8 0.8)) (justify left bottom))
   )
-  (text "Adjust for\nSMD LED!" (at 55.88 78.74 0)
+  (text "180mcd \nor more" (at 46.355 58.42 0)
     (effects (font (size 0.8 0.8)) (justify left bottom))
   )
@@
   (symbol (lib_id "Device:LED") (at 42.545 60.96 90) (unit 1)
     (in_bom no) (on_board yes) (dnp yes)
-    (property "Reference" "D?" (at 46.355 60.96 90)
+    (property "Reference" "D?" (at 37.465 60.96 90)
       (effects (font (size 1.27 1.27)) (justify right))
     )
-    (property "Value" "gn" (at 46.355 63.5 90)
+    (property "Value" "gn" (at 37.465 63.5 90)
       (effects (font (size 1.27 1.27)) (justify right))
     )
-    (property "Footprint" "LED_SMD:LED_0805_2012Metric_Pad1.15x1.40mm_HandSolder" (at 42.545 60.96 0)
+    (property "Footprint" "LED_SMD:LED_0603_1608Metric_Pad1.05x0.95mm_HandSolder" (at 42.545 60.96 0)
       (effects (font (size 1.27 1.27)) hide)
     )
